File: extras/schematic/schematic_basic.sch (EAGLE design)
At the start: 1 part

Commit message: SI47XX Arduino LIbrary
Parts:
- added AM, FM: (no value), discrete:ANTENNA
- added C1: 22nF, SparkFun-Capacitors:22NF/22,000PF-0603-50V-10%
- added C2, C3: 22pF, SparkFun-Capacitors:22PF-0603-50V-5%
- added C4, C5: 4.7uF, SparkFun-Capacitors:4.7UF-1206-16V-(+80/-20%)
- added C6: 100nF, rcl:CXXC10B6
- added CX1, CX2: (no value), rcl:CXXC10B6
- added J1: (no value), SparkFun-Connectors:AUDIO_JACK_2.5MMSPECIAL_POGO_PINS
- added L1: (no value), ngspice-simulation:L
- added R1, R2: 4.7k, SparkFun-Resistors:4.7KOHM-0603-1/10W-1%
- added U1: SI4735-D60-GU, si4735:SI4735-D60-GU
- added Y1: (no value), SparkFun-Clocks:CRYSTALPTH-2X6
Connections:
- new net GND: C2.2, C3.2, C6.1, J1.SLEEVE, L1.1, R1.1, R2.1, U1.!SEN, U1.GND, U1.GND_2, U1.RFGND
- new net N$1: B1.*9, U1.!RST
- new net N$10: AM.1, CX1.2, L1.2
- new net N$12: CX1.1, U1.AMI
- new net N$13: CX2.2, U1.FMI
- new net N$14: CX2.1, FM.1
- new net N$2: B1.A4, R1.2, U1.SCLK
- new net N$3: C2.1, U1.RCLK, Y1.2
- new net N$4: C1.1, U1.DBYP
- new net N$5: C3.1, U1.GPO3/[DCLK], Y1.1
- new net N$6: C5.2, U1.LOUT/[DFS]
- new net N$7: C4.2, U1.ROUT/[DOUT]
- new net N$8: C5.1, J1.LEFT
- new net N$9: C4.1, J1.RIGHT
- new net SDA: B1.A5, R2.2, U1.SDIO
- new net VCC: C1.2, C6.2, U1.VA, U1.VD
Other:
- moved on the sheet: B1

Commit message: SI47XX Arduino Library
Parts:
- removed CX1, CX2: (no value), rcl:CXXC10B6
- added C7, C8: 4.7uF, SparkFun-Capacitors:4.7UF-1206-16V-(+80/-20%)
- added R3: 2.2k, SparkFun-Resistors:2.2KOHM-0603-1/10W-1%
- C2, C3: value 22pF -> (none); device SparkFun-Capacitors:22PF-0603-50V-5% -> rcl:CXXC10B6
- C4: value 4.7uF -> 100nF; device SparkFun-Capacitors:4.7UF-1206-16V-(+80/-20%) -> rcl:CXXC10B6
- C5: value 4.7uF -> 22pF; device SparkFun-Capacitors:4.7UF-1206-16V-(+80/-20%) -> SparkFun-Capacitors:22PF-0603-50V-5%
- C6: value 100nF -> 22pF; device rcl:CXXC10B6 -> SparkFun-Capacitors:22PF-0603-50V-5%
- renumbered R1 to R4, R2 to R5
Connections:
- new net N$11: C5.1, R3.2, Y1.1
- net GND: now also B1.GND@2, C4.1, C5.2, C6.2; no longer C2.2, C3.2, C6.1
- net N$10: now also C3.2; no longer CX1.2
- net N$12: now also C3.1; no longer CX1.1
- net N$13: now also C2.2; no longer CX2.2
- net N$14: now also C2.1; no longer CX2.1
- net N$3: now also C6.1; no longer C2.1
- net N$5: now also R3.1; no longer C3.1, Y1.1
- net N$6: now also C7.2; no longer C5.2
- net N$7: now also C8.2; no longer C4.2
- net N$8: now also C7.1; no longer C5.1
- net N$9: now also C8.1; no longer C4.1
- net VCC: now also B1.VCC, C4.2; no longer C6.2
Other:
- moved on the sheet: C2, C3, C4, C5, C6

Commit message: SI47XX Arduino Library
Connections:
- net GND: now also U1.NC, U1.NC_4
Changed lines of the file:
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@@
 <part name="GND6" library="supply1" library_urn="urn:adsk.eagle:library:371" deviceset="GND" device=""/>
 <part name="SUPPLY2" library="supply2" library_urn="urn:adsk.eagle:library:372" deviceset="VCC" device=""/>
+<part name="GND7" library="supply1" library_urn="urn:adsk.eagle:library:371" deviceset="GND" device=""/>
 </parts>
 <sheets>
@@
 <attribute name="VALUE" x="107.315" y="111.125" size="1.778" layer="96" rot="R270"/>
 </instance>
+<instance part="GND7" gate="1" x="-58.42" y="86.36" smashed="yes">
+<attribute name="VALUE" x="-60.96" y="83.82" size="1.778" layer="96"/>
+</instance>
 </instances>
 <busses>
@@
 <wire x1="88.9" y1="116.84" x2="101.6" y2="116.84" width="0.1524" layer="91"/>
 </segment>
+<segment>
+<pinref part="U1" gate="A" pin="NC_4"/>
+<pinref part="U1" gate="A" pin="NC"/>
+<wire x1="-33.02" y1="93.98" x2="-33.02" y2="91.44" width="0.1524" layer="91"/>
+<wire x1="-33.02" y1="91.44" x2="-58.42" y2="91.44" width="0.1524" layer="91"/>
+<junction x="-33.02" y="91.44"/>
+<pinref part="GND7" gate="1" pin="GND"/>
+<wire x1="-58.42" y1="91.44" x2="-58.42" y2="88.9" width="0.1524" layer="91"/>
+<junction x="-33.02" y="93.98"/>
+</segment>
 </net>
