File: extras/schematic/schematic_basic.sch (EAGLE design)
At the start: 19 parts, among them U1 SI4735-D60-GU

Commit message: SI473X Arduino Library
Other:
- note added: "Optional"
Changed lines of the file:
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@@
 <text x="22.86" y="55.88" size="1.778" layer="91">If GND, I2C addr =  0x11</text>
 <text x="22.86" y="50.8" size="1.778" layer="91">If VCC, I2C addr =  0x63</text>
+<rectangle x1="-35.56" y1="137.16" x2="-20.32" y2="149.86" layer="205"/>
+<text x="-33.02" y="152.4" size="1.778" layer="205">Optional</text>
 </plain>
 <instances>
