File: extras/schematic/schematic_basic_oled.sch (EAGLE design)
At the start: 18 parts, among them U1 SI4735-D60-GU

Commit message: SI47XX Arduino Library
Parts:
- added BFO: 62P16-HX, rotary-encoder:62P16-HX
- added S1: AVC, switch-dil:DS01E
- added S2: Bandwidth, switch-dil:DS01E
- added S3: Band Up, switch-dil:DS01E
- added S4: Band Down, switch-dil:DS01E
- added S5: Vol Up, switch-dil:DS01E
- added S6: Vol Down, switch-dil:DS01E
- added U$1: DISPLAY-OLED-128X64-I2C, diy-modules:DISPLAY-OLED-128X64-I2C
Connections:
- new net N$15: B1.2, BFOA.A
- new net N$16: B1.*3, BFOA.B
- new net N$17: B1.4, S6.1
- new net N$18: B1.*5, S5.1
- new net N$19: B1.*6, S4.1
- new net N$20: B1.7, S3.1
- new net N$21: B1.8, S2.1
- new net N$22: B1.*9, S1.1
- new net N$24: B1.13, BFOSW.E
- net GND: now also BFOA.GND, BFOSW.D, S1.2, S2.2, S3.2, S4.2, S5.2, S6.2, U$1.GND
- net N$2: now also R5.2, U$1.SDA; no longer R4.2
- net SDA: now also R4.2, U$1.SCL; no longer R5.2
- net VCC: now also U$1.VCC
Other:
- moved on the sheet: AM, B1, C1, C2, C3, C4, C5, C6, C7, C8, FM, J1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

Commit message: SI47XX Arduino Library
Connections:
- net GND: no longer R4.1, R5.1, U$1.GND
- net VCC: now also R4.1, R5.1, U$1.GND
Changed lines of the file:
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@@
 <part name="R4" library="SparkFun-Resistors" library_urn="urn:adsk.eagle:library:532" deviceset="4.7KOHM" device="-0603-1/10W-1%" package3d_urn="urn:adsk.eagle:package:39650/1" value="4.7k"/>
 <part name="R5" library="SparkFun-Resistors" library_urn="urn:adsk.eagle:library:532" deviceset="4.7KOHM" device="-0603-1/10W-1%" package3d_urn="urn:adsk.eagle:package:39650/1" value="4.7k"/>
-<part name="GND2" library="supply1" library_urn="urn:adsk.eagle:library:371" deviceset="GND" device=""/>
 <part name="SUPPLY1" library="supply2" library_urn="urn:adsk.eagle:library:372" deviceset="VCC" device=""/>
 <part name="C1" library="SparkFun-Capacitors" library_urn="urn:adsk.eagle:library:510" deviceset="22NF/22,000PF" device="-0603-50V-10%" package3d_urn="urn:adsk.eagle:package:37414/1" value="22nF"/>
@@
 <part name="S6" library="switch-dil" library_urn="urn:adsk.eagle:library:375" deviceset="DS01E" device="" package3d_urn="urn:adsk.eagle:package:27201/2" value="Vol Down"/>
 <part name="GND8" library="supply1" library_urn="urn:adsk.eagle:library:371" deviceset="GND" device=""/>
+<part name="SUPPLY4" library="supply2" library_urn="urn:adsk.eagle:library:372" deviceset="VCC" device=""/>
 </parts>
 <sheets>
@@
 <attribute name="VALUE" x="-8.636" y="121.92" size="1.778" layer="96" font="vector" rot="R270" align="top-center"/>
 </instance>
-<instance part="GND2" gate="1" x="-17.78" y="109.22" smashed="yes">
-<attribute name="VALUE" x="-20.32" y="106.68" size="1.778" layer="96"/>
-</instance>
 <instance part="SUPPLY1" gate="G$1" x="-35.56" y="160.02" smashed="yes" rot="R270">
 <attribute name="VALUE" x="-32.385" y="159.385" size="1.778" layer="96"/>
@@
 <instance part="GND8" gate="1" x="-101.6" y="233.68" smashed="yes">
 <attribute name="VALUE" x="-104.14" y="231.14" size="1.778" layer="96"/>
+</instance>
+<instance part="SUPPLY4" gate="G$1" x="-17.78" y="101.6" smashed="yes" rot="R180">
+<attribute name="VALUE" x="-15.875" y="98.425" size="1.778" layer="96" rot="R180"/>
 </instance>
 </instances>
@@
 <junction x="-53.34" y="142.24"/>
 <junction x="-53.34" y="147.32"/>
-</segment>
-<segment>
-<pinref part="R4" gate="G$1" pin="1"/>
-<pinref part="GND2" gate="1" pin="GND"/>
-<wire x1="-22.86" y1="116.84" x2="-17.78" y2="116.84" width="0.1524" layer="91"/>
-<wire x1="-17.78" y1="116.84" x2="-17.78" y2="111.76" width="0.1524" layer="91"/>
-<pinref part="R5" gate="G$1" pin="1"/>
-<wire x1="-12.7" y1="116.84" x2="-17.78" y2="116.84" width="0.1524" layer="91"/>
-<junction x="-17.78" y="116.84"/>
-<pinref part="U$1" gate="G$1" pin="GND"/>
-<wire x1="5.08" y1="116.84" x2="-17.78" y2="116.84" width="0.1524" layer="91"/>
 </segment>
 <segment>
@@
 <wire x1="38.1" y1="162.56" x2="40.64" y2="162.56" width="0.1524" layer="91"/>
 </segment>
+<segment>
+<pinref part="R4" gate="G$1" pin="1"/>
+<wire x1="-22.86" y1="116.84" x2="-17.78" y2="116.84" width="0.1524" layer="91"/>
+<wire x1="-17.78" y1="116.84" x2="-17.78" y2="111.76" width="0.1524" layer="91"/>
+<pinref part="R5" gate="G$1" pin="1"/>
+<wire x1="-12.7" y1="116.84" x2="-17.78" y2="116.84" width="0.1524" layer="91"/>
+<junction x="-17.78" y="116.84"/>
+<pinref part="U$1" gate="G$1" pin="GND"/>
+<wire x1="5.08" y1="116.84" x2="-17.78" y2="116.84" width="0.1524" layer="91"/>
+<pinref part="SUPPLY4" gate="G$1" pin="VCC"/>
+<wire x1="-17.78" y1="104.14" x2="-17.78" y2="116.84" width="0.1524" layer="91"/>
+</segment>
 </net>
