File: extras/schematic/schematic_basic_oled.sch (EAGLE design)
At the start: 26 parts, among them U1 SI4735-D60-GU

Commit message: SI47XX Arduino Library
Connections:
- net N$24: now also B1.A0; no longer B1.13
Other:
- note added: "A0 = digital pin 14"
Changed lines of the file:
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@@
 <sheet>
 <plain>
+<text x="55.88" y="165.1" size="1.778" layer="91" rot="R90">A0 = digital pin 14</text>
 </plain>
 <instances>
@@
 <segment>
 <pinref part="BFO" gate="SW" pin="E"/>
-<wire x1="27.94" y1="215.9" x2="50.8" y2="215.9" width="0.1524" layer="91"/>
-<wire x1="50.8" y1="215.9" x2="50.8" y2="149.86" width="0.1524" layer="91"/>
-<pinref part="B1" gate="G$1" pin="13"/>
-<wire x1="50.8" y1="149.86" x2="38.1" y2="149.86" width="0.1524" layer="91"/>
-</segment>
-</net>
+<wire x1="27.94" y1="215.9" x2="58.42" y2="215.9" width="0.1524" layer="91"/>
+<wire x1="58.42" y1="215.9" x2="58.42" y2="152.4" width="0.1524" layer="91"/>
+<pinref part="B1" gate="G$1" pin="A0"/>
+<wire x1="58.42" y1="152.4" x2="38.1" y2="152.4" width="0.1524" layer="91"/>
+</segment>
+</net>

Commit message: SI473X Arduino Library
Other:
- note added: "Optional"
Changed lines of the file:
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@@
 <plain>
 <text x="55.88" y="165.1" size="1.778" layer="91" rot="R90">A0 = digital pin 14</text>
+<rectangle x1="-121.92" y1="187.96" x2="-106.68" y2="198.12" layer="205"/>
+<text x="-119.38" y="200.66" size="1.778" layer="205">Optional</text>
 </plain>
 <instances>
