File: extras/schematic/schematic_basic_tft.sch (EAGLE design)
At the start: 26 parts, among them U1 SI4735-D60-GU

Commit message: SI473X Arduino Library
Other:
- note added: "Optional"
Changed lines of the file:
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@@
 <sheet>
 <plain>
+<rectangle x1="-119.38" y1="185.42" x2="-106.68" y2="200.66" layer="205"/>
+<text x="-116.84" y="203.2" size="1.778" layer="205">Optional</text>
 </plain>
 <instances>
