File: extras/schematic/SI4735.brd (EAGLE design)
At the start: 53.3 x 59.7 mm, 20 parts, among them U2 SI4735, Y1 32.768kHz

Commit message: SI47XX Arduino Library
Parts:
- Y1: device SparkFun:CRYSTAL-32KHZ-SMD -> SparkFun:CRYSTAL-32kHz-SMD
Changed lines of the file:
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@@
 <attribute name="VALUE" x="19.812" y="49.657" size="0.4064" layer="27" rot="R180"/>
 </element>
-<element name="Y1" library="SparkFun" package="CRYSTAL-32KHZ-SMD" value="32.768kHz" x="33.02" y="40.64" smashed="yes" rot="R270">
+<element name="Y1" library="SparkFun" package="CRYSTAL-32kHz-SMD" value="32.768kHz" x="33.02" y="40.64" smashed="yes" rot="R270">
 <attribute name="NAME" x="41.275" y="41.275" size="0.4064" layer="25" rot="R270"/>
 <attribute name="VALUE" x="31.115" y="41.275" size="0.4064" layer="27" rot="R270"/>
