File: extras/schematic/schematic_minimal_circuit_with_LCD_16x2_3_3V.sch (EAGLE design)
At the start: 26 parts, among them U1 SI4735-D60-GU

Commit message: SI47XX Arduino Library
Parts:
- removed B1: ARDUINO_PRO_MINI, SparkFun-Boards:ARDUINO_PRO_MINI
- removed BFO: 62P16-HX, rotary-encoder:62P16-HX
- removed S2: Bandwidth, switch-dil:DS01E
- removed S3: Band Up, switch-dil:DS01E
- removed S4: Band Down, switch-dil:DS01E
- removed S5: Vol Up, switch-dil:DS01E
- removed S6: Vol Down, switch-dil:DS01E
- removed U$1: DISPLAY-OLED-128X64-I2C, diy-modules:DISPLAY-OLED-128X64-I2C
- added C10, C9: 22pF, SparkFun-Capacitors:22PF-0603-50V-5%
- added LCD1, LCD2: LCD-16X2SILK, SparkFun-Displays:LCD-16X2SILK
- added R1: 10k, SparkFun-Resistors:10KOHM-0603-1/10W-1%
- added R2: 3.3k, SparkFun-Resistors:3.3KOHM-0603-1/10W-1%
- added U2: 328P, SparkFun-IC-Microcontroller:ATMEGA328P_PDIP
- added Y2: 12MHz, SparkFun-Clocks:CRYSTAL-12MHZ"
- R4: value 4.7k -> 3.3k; device SparkFun-Resistors:4.7KOHM-0603-1/10W-1% -> SparkFun-Resistors:3.3KOHM-0603-1/10W-1%
- R5: value 4.7k -> 1.5k; device SparkFun-Resistors:4.7KOHM-0603-1/10W-1% -> SparkFun-Resistors:1.5KOHM-0603-1/10W-1%
- S1: value AVC -> TL36WO; device switch-dil:DS01E -> switch:TL36WO
Connections:
- removed net N$24: B1.13, BFOSW.E
- removed net SDA: B1.A5, R4.2, U$1.SCL, U1.SCLK
- new net N$23: LCD1.DB4, LCD2.DB4, U2.PD7(AIN1)
- new net N$25: LCD1.DB0, LCD2.DB0
- new net N$26: LCD1.DB1, LCD2.DB1
- new net N$27: LCD1.DB2, LCD2.DB2
- new net N$28: LCD1.DB3, LCD2.DB3
- new net N$29: LCD1.E, LCD2.E, U2.PB5(SCK)
- new net N$32: LCD1.RS, LCD2.RS, U2.PB4(MISO)
- new net N$34: LCD1.VO, LCD2.VO, R5.1
- net GND: now also C10.2, C9.2, LCD1.K, LCD1.VSS, LCD2.K, LCD2.VSS, R5.2, S1.O, U2.GND@1, U2.GND@2; no longer B1.GND@2, BFOA.GND, BFOSW.D, S1.2, S2.2, S3.2, S4.2, S5.2, S6.2, U1.!SEN
- net N$1: now also R1.1, U2.PC6(/RESET); no longer B1.12, U1.!RST
- net N$15: now also R4.2, U1.SCLK, U2.PC5(ADC5/SCL); no longer B1.2, BFOA.A
- net N$16: now also C9.1, U2.PB6(XTAL1/TOSC1), Y2.2; no longer B1.*3, BFOA.B
- net N$17: now also C10.1, U2.PB7(XTAL2/TOSC2), Y2.1; no longer B1.4, S6.1
- net N$18: now also R2.1, U1.SDIO, U2.PC4(ADC4/SDA); no longer B1.*5, S5.1
- net N$19: now also LCD1.DB7, LCD2.DB7, U2.PD4(XCK/T0); no longer B1.*6, S4.1
- net N$2: now also S1.P, U1.!SEN; no longer B1.A4, R5.2, U$1.SDA, U1.SDIO
- net N$20: now also U1.!RST, U2.PB1(OC1A); no longer B1.7, S3.1
- net N$21: now also LCD1.DB6, LCD2.DB6, U2.PD5(T1); no longer B1.8, S2.1
- net N$22: now also LCD1.DB5, LCD2.DB5, U2.PD6(AIN0); no longer B1.*9, S1.1
- net VCC: now also LCD1.A, LCD1.R/W, LCD1.VDD, LCD2.A, LCD2.R/W, LCD2.VDD, R1.2, R2.2, S1.S, U2.VCC; no longer B1.VCC, R5.1, U$1.GND, U$1.VCC
Other:
- note added: "ATMEGA328, Standalone, 12MHz, 3.3V"
- note added: "Based on Mirko Pavleski project"
- note added: "D12"
- note added: "D13"
- note added: "D4"
- note added: "D5"
- note added: "D6"
- note added: "D7"
- note added: "D9"
- note added: "If GND, I2C addr = 0x11"
- note added: "If VCC, I2C addr = 0x63"
- note added: "VCC = 3.3V"
- moved on the sheet: AM, C1, C2, C3, C4, C5, C6, C7, C8, FM, J1, L1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
