File: extras/schematic/schematic_basic_oled_SI47XX_02_ALL_IN_ONE_OLED.sch (EAGLE design)
At the start: 28 parts, among them U1 SI4735-D60-GU

Commit message: SI473X Arduino Library
Other:
- note added: "Optional"
Changed lines of the file:
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@@
 <text x="-160.02" y="238.76" size="1.778" layer="91">Sketche: SI47XX_02_ALL_IN_ONE_OLED.ino</text>
 <text x="-160.02" y="246.38" size="1.778" layer="91">SI4735 all in one with SSB Support</text>
+<rectangle x1="-172.72" y1="185.42" x2="-157.48" y2="200.66" layer="205"/>
+<text x="-170.18" y="203.2" size="1.778" layer="205">Optional</text>
 </plain>
 <instances>
