File: extras/schematic/schematic_basic_active_crystal_osc.sch (EAGLE design)
At the start: 15 parts, among them U1 SI4735-D60-GU

Commit message: SI4735 Arduino Library
Other:
- note added: "external clock"
Changed lines of the file:
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@@
 <text x="22.86" y="55.88" size="1.778" layer="91">If GND, I2C addr =  0x11</text>
 <text x="22.86" y="50.8" size="1.778" layer="91">If VCC, I2C addr =  0x63</text>
+<text x="40.64" y="104.14" size="1.778" layer="91">external clock</text>
 </plain>
 <instances>
@@
 <pinref part="U1" gate="A" pin="RCLK"/>
 <wire x1="33.02" y1="104.14" x2="60.96" y2="104.14" width="0.1524" layer="91"/>
-<wire x1="60.96" y1="104.14" x2="60.96" y2="142.24" width="0.1524" layer="91"/>
-</segment>
-</net>
+</segment>
+</net>
