File: extras/schematic/schematic_basic_lilyGO_esp32.sch (EAGLE design)
At the start: 18 parts, among them U1 SI4735-D60-GU

Commit message: Examples
Parts:
- removed ESP32: See your ESP32 pinout, SparkFun-Boards:ESP32_THING_WO_ANT_KEEPOUT
- added U2: ESP32-DEVKITC-32D, ESP32-DEVKITC-32D:ESP32-DEVKITC-32D
Connections:
- net GND: now also U2.GND3; no longer ESP32.GND@21
- net N$1: now also U2.IO16; no longer ESP32.12
- net N$2: now also U2.SD1; no longer ESP32.21
- net SDA: now also U2.IO18; no longer ESP32.19, ESP32.22
- net VCC: no longer ESP32.3V3@5
Changed lines of the file:
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@@
 <part name="R3" library="SparkFun-Resistors" library_urn="urn:adsk.eagle:library:532" deviceset="2.2KOHM" device="-0603-1/10W-1%" package3d_urn="urn:adsk.eagle:package:39650/1" value="2.2k"/>
 <part name="GND7" library="supply1" library_urn="urn:adsk.eagle:library:371" deviceset="GND" device=""/>
-<part name="ESP32" library="SparkFun-Boards" library_urn="urn:adsk.eagle:library:509" deviceset="ESP32_THING" device="_WO_ANT_KEEPOUT" package3d_urn="urn:adsk.eagle:package:37351/1" value="See your ESP32 pinout"/>
 <part name="SUPPLY2" library="supply2" library_urn="urn:adsk.eagle:library:372" deviceset="VCC" device=""/>
 <part name="GND2" library="supply1" library_urn="urn:adsk.eagle:library:371" deviceset="GND" device=""/>
 <part name="SUPPLY3" library="supply2" library_urn="urn:adsk.eagle:library:372" deviceset="VCC" device=""/>
+<part name="U2" library="ESP32-DEVKITC-32D" deviceset="ESP32-DEVKITC-32D" device=""/>
 </parts>
 <sheets>
@@
 <attribute name="VALUE" x="-154.94" y="129.54" size="1.778" layer="96"/>
 </instance>
-<instance part="ESP32" gate="G$1" x="-2.54" y="165.1" smashed="yes">
-<attribute name="NAME" x="-12.7" y="193.294" size="1.778" layer="95" font="vector"/>
-<attribute name="VALUE" x="-15.24" y="136.906" size="1.778" layer="96" font="vector" align="top-left"/>
-</instance>
 <instance part="SUPPLY2" gate="G$1" x="-33.02" y="101.6" smashed="yes" rot="R180">
 <attribute name="VALUE" x="-31.115" y="98.425" size="1.778" layer="96" rot="R180"/>
 </instance>
-<instance part="GND2" gate="1" x="12.7" y="203.2" smashed="yes" rot="R180">
-<attribute name="VALUE" x="15.24" y="205.74" size="1.778" layer="96" rot="R180"/>
-</instance>
-<instance part="SUPPLY3" gate="G$1" x="-20.32" y="154.94" smashed="yes">
-<attribute name="VALUE" x="-22.225" y="158.115" size="1.778" layer="96"/>
+<instance part="GND2" gate="1" x="25.4" y="205.74" smashed="yes" rot="R180">
+<attribute name="VALUE" x="27.94" y="208.28" size="1.778" layer="96" rot="R180"/>
+</instance>
+<instance part="SUPPLY3" gate="G$1" x="-25.4" y="172.72" smashed="yes">
+<attribute name="VALUE" x="-27.305" y="175.895" size="1.778" layer="96"/>
+</instance>
+<instance part="U2" gate="G$1" x="0" y="172.72" smashed="yes">
+<attribute name="NAME" x="-15.2572" y="198.7843" size="1.78" layer="95"/>
+<attribute name="VALUE" x="-15.2563" y="144.7502" size="1.7799" layer="96"/>
 </instance>
 </instances>
@@
 </segment>
 <segment>
-<pinref part="ESP32" gate="G$1" pin="GND@21"/>
-<wire x1="10.16" y1="190.5" x2="12.7" y2="190.5" width="0.1524" layer="91"/>
+<pinref part="U2" gate="G$1" pin="GND3"/>
+<wire x1="20.32" y1="195.58" x2="25.4" y2="195.58" width="0.1524" layer="91"/>
 <pinref part="GND2" gate="1" pin="GND"/>
-<wire x1="12.7" y1="190.5" x2="12.7" y2="200.66" width="0.1524" layer="91"/>
+<wire x1="25.4" y1="195.58" x2="25.4" y2="203.2" width="0.1524" layer="91"/>
 </segment>
 </net>
@@
 <segment>
 <pinref part="R5" gate="G$1" pin="2"/>
-<wire x1="-27.94" y1="129.54" x2="-27.94" y2="127" width="0.1524" layer="91"/>
 <pinref part="U1" gate="A" pin="SDIO"/>
-<wire x1="-27.94" y1="127" x2="-27.94" y2="119.38" width="0.1524" layer="91"/>
+<wire x1="-27.94" y1="129.54" x2="-27.94" y2="124.46" width="0.1524" layer="91"/>
+<wire x1="-27.94" y1="124.46" x2="-27.94" y2="119.38" width="0.1524" layer="91"/>
 <wire x1="-60.96" y1="147.32" x2="-33.02" y2="147.32" width="0.1524" layer="91"/>
 <wire x1="-33.02" y1="147.32" x2="-33.02" y2="129.54" width="0.1524" layer="91"/>
 <wire x1="-33.02" y1="129.54" x2="-27.94" y2="129.54" width="0.1524" layer="91"/>
-<pinref part="ESP32" gate="G$1" pin="22"/>
-<wire x1="10.16" y1="180.34" x2="10.16" y2="177.8" width="0.1524" layer="91"/>
-<wire x1="10.16" y1="177.8" x2="27.94" y2="177.8" width="0.1524" layer="91"/>
-<wire x1="27.94" y1="177.8" x2="27.94" y2="127" width="0.1524" layer="91"/>
-<wire x1="27.94" y1="127" x2="-27.94" y2="127" width="0.1524" layer="91"/>
-<junction x="-27.94" y="127"/>
-<pinref part="ESP32" gate="G$1" pin="19"/>
-<junction x="10.16" y="177.8"/>
+<pinref part="U2" gate="G$1" pin="IO18"/>
+<wire x1="20.32" y1="175.26" x2="27.94" y2="175.26" width="0.1524" layer="91"/>
+<wire x1="27.94" y1="175.26" x2="27.94" y2="124.46" width="0.1524" layer="91"/>
+<wire x1="27.94" y1="124.46" x2="-27.94" y2="124.46" width="0.1524" layer="91"/>
+<junction x="-27.94" y="124.46"/>
 </segment>
 </net>
@@
 <pinref part="U1" gate="A" pin="SCLK"/>
 <wire x1="-60.96" y1="144.78" x2="-38.1" y2="144.78" width="0.1524" layer="91"/>
-<wire x1="-38.1" y1="144.78" x2="-38.1" y2="121.92" width="0.1524" layer="91"/>
-<pinref part="ESP32" gate="G$1" pin="21"/>
-<wire x1="-38.1" y1="121.92" x2="-38.1" y2="119.38" width="0.1524" layer="91"/>
-<wire x1="10.16" y1="187.96" x2="30.48" y2="187.96" width="0.1524" layer="91"/>
-<wire x1="30.48" y1="187.96" x2="30.48" y2="121.92" width="0.1524" layer="91"/>
-<wire x1="30.48" y1="121.92" x2="-38.1" y2="121.92" width="0.1524" layer="91"/>
-<junction x="-38.1" y="121.92"/>
+<wire x1="-38.1" y1="144.78" x2="-38.1" y2="132.08" width="0.1524" layer="91"/>
+<pinref part="U2" gate="G$1" pin="SD1"/>
+<wire x1="-38.1" y1="132.08" x2="-38.1" y2="119.38" width="0.1524" layer="91"/>
+<wire x1="20.32" y1="154.94" x2="25.4" y2="154.94" width="0.1524" layer="91"/>
+<wire x1="25.4" y1="154.94" x2="25.4" y2="132.08" width="0.1524" layer="91"/>
+<wire x1="25.4" y1="132.08" x2="-38.1" y2="132.08" width="0.1524" layer="91"/>
+<junction x="-38.1" y="132.08"/>
 </segment>
 </net>
@@
 <junction x="-33.02" y="104.14"/>
 </segment>
-<segment>
-<pinref part="ESP32" gate="G$1" pin="3V3@5"/>
-<pinref part="SUPPLY3" gate="G$1" pin="VCC"/>
-<wire x1="-15.24" y1="152.4" x2="-20.32" y2="152.4" width="0.1524" layer="91"/>
-</segment>
 </net>
 <net name="N$4" class="0">
@@
 <segment>
 <pinref part="U1" gate="A" pin="!RST"/>
-<wire x1="-60.96" y1="139.7" x2="-25.4" y2="139.7" width="0.1524" layer="91"/>
-<pinref part="ESP32" gate="G$1" pin="12"/>
-<wire x1="-25.4" y1="139.7" x2="-25.4" y2="160.02" width="0.1524" layer="91"/>
-<wire x1="-25.4" y1="160.02" x2="-15.24" y2="160.02" width="0.1524" layer="91"/>
-</segment>
-</net>
+<pinref part="U2" gate="G$1" pin="IO16"/>
+<wire x1="20.32" y1="167.64" x2="30.48" y2="167.64" width="0.1524" layer="91"/>
+<wire x1="30.48" y1="167.64" x2="30.48" y2="139.7" width="0.1524" layer="91"/>
+<wire x1="30.48" y1="139.7" x2="-60.96" y2="139.7" width="0.1524" layer="91"/>
+</segment>
+</net>
